File: hw/pcb/led-matrix.kicad_sch (KiCad schematic)
At the start: 130 parts, among them Q1 SSM3K37FSLF, Q10 SSM3K37FSLF, Q2 SSM3K37FSLF, Q3 SSM3K37FSLF, Q4 SSM3K37FSLF, Q5 SSM3K37FSLF, Q6 SSM3K37FSLF, Q7 SSM3K37FSLF, Q8 SSM3K37FSLF, Q9 SSM3K37FSLF

Commit message: chore: updated schematic to have correctly sized current limiting resistors
Parts:
- R10, R11, R12, R13, R14, R15, R6, R7, R8, R9: value R -> 820
Other:
- note added: "These LEDs are the APTD1608LSURCK from Kingbright They work with a forward current as low as 2mA (Vf = 1.75V) Hence the large current limiting resistor... (3.3 - Vf) / 0.002 = 775Ω"
Changed lines of the file:
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@@
 	(title_block
 		(title "LED Matrix")
-		(rev "Rev1")
+		(rev "RevB")
 		(company "Isaac Pawley")
 	)
+	(text "These LEDs are the APTD1608LSURCK from Kingbright\nThey work with a forward current as low as 2mA (Vf = 1.75V)\nHence the large current limiting resistor...\n\n(3.3 - Vf) / 0.002 = 775Ω"
+		(exclude_from_sim no)
+		(at 52.578 50.546 0)
+		(effects
+			(font
+				(size 1.27 1.27)
+			)
+			(justify left)
+		)
+	)
 	(junction
 		(at 194.31 44.45)
@@
 			)
 		)
-		(property "Value" "R"
+		(property "Value" "820"
 			(at 132.08 104.14 90)
 			(show_name no)
@@
 			)
 		)
-		(property "Value" "R"
+		(property "Value" "820"
 			(at 132.08 129.54 90)
 			(show_name no)
@@
 			)
 		)
-		(property "Value" "R"
+		(property "Value" "820"
 			(at 132.08 66.04 90)
 			(show_name no)
@@
 			)
 		)
-		(property "Value" "R"
+		(property "Value" "820"
 			(at 132.08 154.94 90)
 			(show_name no)
@@
 			)
 		)
-		(property "Value" "R"
+		(property "Value" "820"
 			(at 132.08 78.74 90)
 			(show_name no)
@@
 			)
 		)
-		(property "Value" "R"
+		(property "Value" "820"
 			(at 132.08 40.64 90)
 			(show_name no)
@@
 			)
 		)
-		(property "Value" "R"
+		(property "Value" "820"
 			(at 132.08 142.24 90)
 			(show_name no)
@@
 			)
 		)
-		(property "Value" "R"
+		(property "Value" "820"
 			(at 132.08 53.34 90)
 			(show_name no)
@@
 			)
 		)
-		(property "Value" "R"
+		(property "Value" "820"
 			(at 132.08 116.84 90)
 			(show_name no)
@@
 			)
 		)
-		(property "Value" "R"
+		(property "Value" "820"
 			(at 132.08 91.44 90)
 			(show_name no)

Commit message: chore: updated schematics to show true part numbers
Parts:
- D10, D100, D101, D102, D103, D104, D11, D12, D13, D14, D15, D16, D17, D18, D19, D20, D21, D22, D23, D24, D25, D26, D27, D28, D29, D30, D31, D32, D33, D34, D35, D36, D37, D38, D39, D40, D41, D42, D43, D44, D45, D46, D47, D48, D49, D5, D50, D51, D52, D53, D54, D55, D56, D57, D58, D59, D6, D60, D61, D62, D63, D64, D65, D66, D67, D68, D69, D7, D70, D71, D72, D73, D74, D75, D76, D77, D78, D79, D8, D80, D81, D82, D83, D84, D85, D86, D87, D88, D89, D9, D90, D91, D92, D93, D94, D95, D96, D97, D98, D99: PN (none) -> APTD1608LSURCK
- Q1, Q10, Q2, Q3, Q4, Q5, Q6, Q7, Q8, Q9: PN (none) -> SSM3K37FS,LF
- R10, R11, R12, R13, R14, R15, R6, R7, R8, R9: PN (none) -> CRGCQ0603F820R
- R16, R17, R18, R19, R20, R21, R22, R23, R24, R25: PN (none) -> CRGCQ0603F100R
