File: hw/pcb/micro-affirmations.kicad_pcb (KiCad board)
At the start: 2 copper layers, 70 x 40 mm, 157 parts, among them J1 USB-C_2171750001, J2 DEBUG, Q1 SSM3K37FSLF, Q10 SSM3K37FSLF, Q2 SSM3K37FSLF, Q3 SSM3K37FSLF, Q4 SSM3K37FSLF, Q5 SSM3K37FSLF, Q6 SSM3K37FSLF, Q7 SSM3K37FSLF, Q8 SSM3K37FSLF, Q9 SSM3K37FSLF, SW1 SW_Push, U1 STM32C031C6Tx, U2 TPS61094

Commit message: fix: rewired swd pins and supercap changer enable pins
Parts:
- removed D105, D2, D3, D4: TVS, Diode_SMD:D_SOD-923
- added D1: CHARGE, Diode_SMD:D_0603_1608Metric, F.Cu at (123.3, 113.5)
- added G***: LOGO, LOGO, F.Cu at (159.6, 105.2)
- added H1: MountingHole, MountingHole:MountingHole_2.2mm_M2, F.Cu at (116.5, 87.0)
- added JP1: SolderJumper_2_Bridged, Jumper:SolderJumper-2_P1.3mm_Bridged_RoundedPad1.0x1.5mm, F.Cu at (172.3, 111.7)
- added R3: 1.5k, Resistor_SMD:R_0603_1608Metric, F.Cu at (123.3, 117.2)
- added TP2: TestPoint, TestPoint:TestPoint_Pad_D1.0mm, F.Cu at (123.3, 122.2)
- added TP3: TestPoint, TestPoint:TestPoint_Pad_D1.0mm, F.Cu at (175.6, 116.0)
- added TP4: TestPoint, TestPoint:TestPoint_Pad_D1.0mm, F.Cu at (182.3, 107.5)
- added TP5: TestPoint, TestPoint:TestPoint_Pad_D1.0mm, F.Cu at (180.6, 108.9)
- added TP6: TestPoint, TestPoint:TestPoint_Pad_D1.0mm, F.Cu at (180.9, 99.9)
- added TP7: TestPoint, TestPoint:TestPoint_Pad_D1.0mm, B.Cu at (178.4, 97.6)
- added TP8: TestPoint, TestPoint:TestPoint_Pad_D1.0mm, F.Cu at (116.0, 93.2)
- J1: value USB-C_2171750001 -> USBC
- L1: value L -> 2.2u
- Q1, Q10, Q2, Q3, Q4, Q5, Q6, Q7, Q8, Q9: value SSM3K37FSLF -> NCH
- R4: value ~ -> 5.1k
- R5: value ~ -> 10k
- SW1: value SW_Push -> RST
- moved C8 41.6 mm to (174.1, 119.3), turned to -90 degrees
- moved R5 41.5 mm to (163.6, 111.7), turned to -90 degrees
- moved C10 40.9 mm to (165.4, 114.7)
- moved U2 40.9 mm to (168.8, 118.3)
- moved R4 40.5 mm to (163.6, 114.8), turned to -90 degrees
- moved R26 40.1 mm to (167.8, 114.7), turned to -90 degrees
- moved C7 39.6 mm to (172.1, 119.3), turned to -90 degrees
- moved R28 38.4 mm to (169.8, 114.7)
- moved R27 37.4 mm to (171.9, 114.7)
- moved C9 36.6 mm to (168.8, 121.3)
- moved L1 36.1 mm to (164.0, 119.0), turned to 180 degrees
- moved C1 21.0 mm to (159.5, 116.5), turned to 180 degrees
- moved C3 3.03 mm to (179.0, 114.6)
- moved Q4 2.01 mm to (131.4, 100.1), turned to 90 degrees
- moved Q6 2.01 mm to (136.5, 100.1), turned to 90 degrees
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Connections:
- C9 pad 1: +3V3 -> CAP_VOLT
- Q1 pad 1: Net-(D15-K) -> Net-(Q1-G)
- Q1 pad 2: Net-(Q1-G) -> GND
- Q1 pad 3: GND -> Net-(D15-K)
- Q10 pad 1: Net-(D104-K) -> Net-(Q10-G)
- Q10 pad 2: Net-(Q10-G) -> GND
- Q10 pad 3: GND -> Net-(D104-K)
- Q2 pad 1: Net-(D16-K) -> Net-(Q2-G)
- Q2 pad 2: Net-(Q2-G) -> GND
- Q2 pad 3: GND -> Net-(D16-K)
- Q3 pad 1: Net-(D17-K) -> Net-(Q3-G)
- Q3 pad 2: Net-(Q3-G) -> GND
- Q3 pad 3: GND -> Net-(D17-K)
- Q4 pad 1: Net-(D18-K) -> Net-(Q4-G)
- Q4 pad 2: Net-(Q4-G) -> GND
- Q4 pad 3: GND -> Net-(D18-K)
- Q5 pad 1: Net-(D19-K) -> Net-(Q5-G)
- Q5 pad 2: Net-(Q5-G) -> GND
- Q5 pad 3: GND -> Net-(D19-K)
- Q6 pad 1: Net-(D10-K) -> Net-(Q6-G)
- Q6 pad 2: Net-(Q6-G) -> GND
- Q6 pad 3: GND -> Net-(D10-K)
- Q7 pad 1: Net-(D101-K) -> Net-(Q7-G)
- Q7 pad 2: Net-(Q7-G) -> GND
- Q7 pad 3: GND -> Net-(D101-K)
- Q8 pad 1: Net-(D102-K) -> Net-(Q8-G)
- Q8 pad 2: Net-(Q8-G) -> GND
- Q8 pad 3: GND -> Net-(D102-K)
- Q9 pad 1: Net-(D103-K) -> Net-(Q9-G)
- Q9 pad 2: Net-(Q9-G) -> GND
- Q9 pad 3: GND -> Net-(D103-K)
- U1 pad 1: /DEBUG_SWDIO -> Net-(U1-PC13)
- U1 pad 11: unconnected-(U1-PA0-Pad11) -> Net-(U1-PA0)
- U1 pad 2: /DEBUG_SWCLK -> unconnected-(U1-PC14-Pad2)
- U1 pad 35: unconnected-(U1-PA13-Pad35) -> /DEBUG_SWDIO
- U1 pad 36: unconnected-(U1-PA14-Pad36) -> /DEBUG_SWCLK
- U1 pad 45: unconnected-(U1-PB6-Pad45) -> Net-(U1-PB6)
- U1 pad 48: unconnected-(U1-PB9-Pad48) -> Net-(U1-PB9)
- U2 pad 13: unconnected-(U2-Pad13) -> GND
- U2 pad 2: +5V -> Net-(JP1-B)
- U2 pad 3: +5V -> Net-(JP1-B)
Routing:
- net +3V3: track 91.6 -> 28.4 mm
- net /CHARGE_SENSE: track 79.5 -> 28.3 mm
- net +5V: track 23.3 -> 63.2 mm
- net CAP_VOLT: track 78.5 -> 41.0 mm, vias 0 -> 3
- net /DEBUG_SWDIO: track 10.1 -> 23.3 mm, vias 0 -> 1
- net /DEBUG_SWCLK: track 12.9 -> 24.3 mm, vias 0 -> 1
- net Net-(JP1-B): track 0.00 -> 10.9 mm
- net Net-(U2-SW): track 5.40 -> 0.00 mm
- net Net-(U1-PC13): track 0.00 -> 3.55 mm
- net Net-(U1-PB6): track 0.00 -> 3.18 mm
- net Net-(U1-PB9): track 0.00 -> 3.09 mm
- net Net-(U2-ICHG): track 5.95 -> 3.21 mm
- net Net-(U1-PA0): track 0.00 -> 2.30 mm, vias 0 -> 1
- net Net-(D1-A): track 0.00 -> 2.07 mm
- net Net-(D18-K): track 58.0 -> 56.0 mm
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