File: hw/pcb/micro-affirmations.kicad_sch (KiCad schematic)
At the start: 16 parts, among them J1 USB-C_2171750001, J2 DEBUG, SW1 SW_Push, U1 STM32C031C6Tx

Commit message: fix: rewired swd pins and supercap changer enable pins
Parts:
- removed D105, D2, D3, D4: TVS, Diode_SMD:D_SOD-923, symbol Device:D_Zener
- added D1: CHARGE, Diode_SMD:D_0603_1608Metric, symbol Device:LED
- added H1: MountingHole, MountingHole:MountingHole_2.2mm_M2, symbol Mechanical:MountingHole
- added R3: 1.5k, Resistor_SMD:R_0603_1608Metric, symbol Device:R
- added TP2, TP4, TP5, TP6, TP7, TP8: TestPoint, TestPoint:TestPoint_Pad_D1.0mm, symbol Connector:TestPoint
- J1: value USB-C_2171750001 -> USBC
- J2: now left out of the parts list
- SW1: value SW_Push -> RST
Connections:
- net +5V: now also R3.1, TP2.1
- net DEBUG_SWCLK: now also U1.36 (PA14); no longer U1.2 (PC14)
- net DEBUG_SWDIO: now also U1.35 (PA13); no longer U1.1 (PC13)
- net GND: now also D1.1 (K), TP8.1
- net at U1.11 (PA0): now also TP7.1
- net at U1.45 (PB6): now also TP5.1
- net at U1.48 (PB9): now also TP4.1
- new net: TP6.1, U1.1 (PC13)
- new net: D1.2 (A), R3.2
- no-connect marks 20 -> 1
Other:
- moved on the sheet: J2, R4, R5
